File: PCB/CueTracker/CueTracker.kicad_sch (KiCad schematic)
At the start: 153 parts, among them J1 USB4105-GF-A, J2 JTAG/RECOVERY, Q1 CSD87313DMS, SW1 SHIP EXIT, U1 TUSB320LAI, U10 BQ298217, U11 IIS3DWB10ISTR, U12 LSM6DSV320XTR, U13 TLV320ADC6120IRTER, U14 BQ27427, U2 USBLC6-2SC6, U3 ESP32-S3R8, U4 W25Q128JVSIQ, U5 TPS63802DLAR, U6 BMP581, U7 BQ25611D, U8 MMC5983MA, U9 TPS22919, Y1 40MHz, Y2 32.768kHz

Commit message: pcb: migrate CueTracker to split PICO architecture
Parts:
- removed AE1: CA-C03, CueTracker_Exact:CA-C03_2.4GHz_Chip_Antenna, symbol CueTracker_Exact:CA-C03
- removed BOOT1: SW_BOOT, Button_Switch_SMD:SW_SPST_EVQP2_MiddlePushTravel_H2.5mm, symbol Switch:SW_Push
- removed BT1: 1S 18650 / 21700, Connector_Wire:SolderWire-0.5sqmm_1x02_P4.8mm_D0.9mm_OD2.3mm_Relief2x, symbol Device:Battery_Cell
- removed C1, C10, C11, C34, C35, C36, C40, C41, C44, C46, C48, C49, C51, C54, C56, C57: 100n, Capacitor_SMD:C_0402_1005Metric, symbol Device:C_Small
- removed C12, C15, C16, C3, C33, C4, C5, C6, C8: 100n, Capacitor_SMD:C_0402_1005Metric_Pad0.74x0.62mm_HandSolder, symbol Device:C_Small
- removed C13, C21: 22u, Capacitor_SMD:C_0805_2012Metric, symbol Device:C_Small
- removed C14, C18: 10u, Capacitor_SMD:C_0402_1005Metric_Pad0.74x0.62mm_HandSolder, symbol Device:C_Small
- removed C17, C32: 10u, Capacitor_SMD:C_0603_1608Metric, symbol Device:C_Small
- removed C19, C20: 1p5, Capacitor_SMD:C_0201_0603Metric, symbol Device:C_Small
- removed C2, C7, C9: 1u, Capacitor_SMD:C_0402_1005Metric_Pad0.74x0.62mm_HandSolder, symbol Device:C_Small
- removed C22, C39, C47, C52, C55, C58, C59: 1u, Capacitor_SMD:C_0603_1608Metric, symbol Device:C_Small
- removed C23: 47n, Capacitor_SMD:C_0402_1005Metric, symbol Device:C_Small
- removed C24, C27, C38, C42, C43, C45: 10u, Capacitor_SMD:C_0805_2012Metric, symbol Device:C_Small
- removed C25: 4u7, Capacitor_SMD:C_0603_1608Metric, symbol Device:C_Small
- removed C26, C37, C50: 1u, Capacitor_SMD:C_0402_1005Metric, symbol Device:C_Small
- removed C28, C29: 16p, Capacitor_SMD:C_0402_1005Metric_Pad0.74x0.62mm_HandSolder, symbol Device:C_Small
- removed C30, C31: 10p, Capacitor_SMD:C_0402_1005Metric_Pad0.74x0.62mm_HandSolder, symbol Device:C_Small
- removed C53: 2u2, Capacitor_SMD:C_0603_1608Metric, symbol Device:C_Small
- removed D1, D2: XL-1005SURC, LED_SMD:LED_0402_1005Metric_Pad0.77x0.64mm_HandSolder, symbol Device:LED
- removed FB1: BLM18KG601SN1D, Inductor_SMD:L_0603_1608Metric, symbol Device:FerriteBead_Small
- removed J1: USB4105-GF-A, Connector_USB:USB_C_Receptacle_GCT_USB4105-xx-A_16P_TopMnt_Horizontal, symbol Connector:USB_C_Receptacle_USB2.0_16P
- removed J2: JTAG/RECOVERY, Connector_PinHeader_1.27mm:PinHeader_2x05_P1.27mm_Vertical_SMD, symbol Connector_Generic:Conn_02x05_Odd_Even
- removed JP1: GAUGE BYPASS, Jumper:SolderJumper-2_P1.3mm_Open_Pad1.0x1.5mm, symbol Jumper:SolderJumper_2_Open
- removed L1: 2n2, Inductor_SMD:L_0603_1608Metric_Pad1.05x0.95mm_HandSolder, symbol Device:L
- removed L2: 470n, Inductors SMD:IND_COILCRAFT_XFL4015, symbol Device:L
- removed L3: 2n4, Inductor_SMD:L_0201_0603Metric, symbol Device:L
- removed L4: 1uH, CueTracker_Exact:L_Eaton_MPI4020V2_4.2x4.4mm_H2.0_Pad2.3x1.65_P3.30mm, symbol Device:L
- removed L5: 24nH, Inductor_SMD:L_0402_1005Metric, symbol Device:L_Small
- removed LED1: WS2812B-2020-V6, LED_SMD:LED_WS2812B-2020_PLCC4_2.0x2.0mm, symbol LED:WS2812B-2020
- removed MK1: IM73A135V01, Sensor_Audio:Infineon_PG-LLGA-5-2, symbol Sensor_Audio:IM73A135V01
- removed Q1: CSD87313DMS, CueTracker_Exact:TI_CSD87313DMS_DMS8_3.3x3.3mm, symbol CueTracker_Exact:CSD87313DMS
- removed R1, R2: 4.7k, Resistor_SMD:R_0402_1005Metric, symbol Device:R_Small
- removed R10: 511k, Resistor_SMD:R_0402_1005Metric_Pad0.72x0.64mm_HandSolder, symbol Device:R_Small
- removed R11, R27, R32, R34, R36, R38: 0R, Resistor_SMD:R_0402_1005Metric, symbol Device:R_Small
- removed R12, R19, R25: 100k, Resistor_SMD:R_0402_1005Metric, symbol Device:R_Small
- removed R13, R17, R18, R20, R26, R28, R45, R8: 10k, Resistor_SMD:R_0402_1005Metric, symbol Device:R_Small
- removed R14: 91k, Resistor_SMD:R_0402_1005Metric_Pad0.72x0.64mm_HandSolder, symbol Device:R_Small
- removed R15, R16, R4, R7: 10k, Resistor_SMD:R_0402_1005Metric_Pad0.72x0.64mm_HandSolder, symbol Device:R_Small
- removed R21: 5.30k, Resistor_SMD:R_0402_1005Metric, symbol Device:R_Small
- removed R22: 31.2k, Resistor_SMD:R_0402_1005Metric, symbol Device:R_Small
- removed R23: 1M, Resistor_SMD:R_0402_1005Metric, symbol Device:R_Small
- removed R24: 330k, Resistor_SMD:R_0402_1005Metric, symbol Device:R_Small
- removed R29, R35, R40, R42, R5, R6: 22R, Resistor_SMD:R_0402_1005Metric, symbol Device:R_Small
- removed R3: 900k, Resistor_SMD:R_0402_1005Metric, symbol Device:R_Small
- removed R30: 300, Resistor_SMD:R_0402_1005Metric, symbol Device:R_Small
- removed R31: 20, Resistor_SMD:R_0402_1005Metric, symbol Device:R_Small
- removed R33: 2k, Resistor_SMD:R_0402_1005Metric, symbol Device:R_Small
- removed R37: 33R, Resistor_SMD:R_0402_1005Metric, symbol Device:R_Small
- removed R39, R43: 0R, Resistor_SMD:R_0603_1608Metric, symbol Device:R_Small
- removed R41: 100R, Resistor_SMD:R_0402_1005Metric, symbol Device:R_Small
- removed R44: 60m, CueTracker_Exact:Vishay_WSL2512_6.35x3.18_P5.71mm_Pad1.65x3.68mm, symbol Device:R_Small
- removed R9: 0R, Resistor_SMD:R_0402_1005Metric_Pad0.72x0.64mm_HandSolder, symbol Device:R_Small
- removed RST1: SW_RST, Button_Switch_SMD:SW_SPST_EVQP2_MiddlePushTravel_H2.5mm, symbol Switch:SW_Push
- removed SW1: SHIP EXIT, Button_Switch_SMD:SW_SPST_PTS810, symbol Switch:SW_Push
- removed TH1: REMOTE 10k NTC PADS, Connector_Wire:SolderWire-0.15sqmm_1x02_P4mm_D0.5mm_OD1.5mm_Relief2x, symbol Device:Thermistor_NTC
- removed TP1, TP2, TP3, TP4, TP5, TP6, TP7, TP8, TP9: TestPoint, TestPoint:TestPoint_Pad_D1.0mm, symbol Connector:TestPoint
- removed TP10: IMPACT_INT1, TestPoint:TestPoint_Pad_D1.0mm, symbol Connector:TestPoint
- removed TP11: IMPACT_INT2, TestPoint:TestPoint_Pad_D1.0mm, symbol Connector:TestPoint
- removed TP12: MOTION_INT1, TestPoint:TestPoint_Pad_D1.0mm, symbol Connector:TestPoint
- removed TP13: MOTION_INT2, TestPoint:TestPoint_Pad_D1.0mm, symbol Connector:TestPoint
- removed U1: TUSB320LAI, CueTracker_Exact:TI_RWB0012A_X2QFN12_1.6x1.6mm_P0.4mm, symbol CueTracker_Exact:TUSB320LAIRWBR
- removed U10: BQ298217, CueTracker_Exact:TI_RUG0008A_X2QFN8_1.5x1.5mm_P0.5mm, symbol CueTracker_Exact:BQ298217RUGR
- removed U11: IIS3DWB10ISTR, CueTracker_Exact:IIS3DWB10IS_LLGA16_4.5x4.5_WF, symbol CueTracker_Exact:IIS3DWB10ISTR
- removed U12: LSM6DSV320XTR, Package_LGA:LGA-14_3x2.5mm_P0.5mm_LayoutBorder3x4y, symbol CueTracker_Exact:LSM6DSV320XTR
- removed U13: TLV320ADC6120IRTER, CueTracker_Exact:TI_RTE0020A_WQFN20_3x3_P0.5_EP1.4, symbol CueTracker_Exact:TLV320ADC6120IRTER_EXACT
- removed U14: BQ27427, CueTracker_Exact:TI_YZF0009_DSBGA9_1.62x1.58mm_P0.5mm, symbol CueTracker_Exact:BQ27427YZFR
- removed U2: USBLC6-2SC6, Package_TO_SOT_SMD:SOT-23-6, symbol Power_Protection:USBLC6-2SC6
- removed U3: ESP32-S3R8, Package_DFN_QFN:QFN-56-1EP_7x7mm_P0.4mm_EP4x4mm, symbol MCU_Espressif:ESP32-S3
- removed U4: W25Q128JVSIQ, Package_SO:SOIC-8_5.3x5.3mm_P1.27mm, symbol Memory_Flash:W25Q128JVS
- removed U5: TPS63802DLAR, CueTracker_Exact:TPS63802_DLA0010A_VSON-HR-10, symbol CueTracker_Exact:TPS63802DLAR
- removed U6: BMP581, CueTracker_Exact:BMP581_LGA10_2x2mm, symbol CueTracker_Exact:BMP581
- removed U7: BQ25611D, CueTracker_Exact:TI_RTW0024A_WQFN24_4x4mm_P0.5mm_EP2.6mm, symbol CueTracker_Exact:BQ25611DRTWR
- removed U8: MMC5983MA, CueTracker_Exact:MMC5983MA_LGA16_3x3mm, symbol CueTracker_Exact:MMC5983MA
- removed U9: TPS22919, CueTracker_Exact:TI_DCK0006A_SC70-6_2.0x1.25mm_P0.65mm, symbol CueTracker_Exact:TPS22919DCKR
- removed Y1: 40MHz, Crystal:Crystal_SMD_3225-4Pin_3.2x2.5mm, symbol Device:Crystal_GND24
- removed Y2: 32.768kHz, Crystal:Crystal_SMD_3215-2Pin_3.2x1.5mm, symbol Device:Crystal
Connections:
- no-connect marks 25 -> 0
Other:
- added sheet Front Sensor (front_sensor.kicad_sch)
- added sheet Rear Main (rear_main.kicad_sch)
- note added: "CueTracker hierarchical partition: rear electronics / front inertial sensors"
- note removed: "10-pin JTAG header"
- note removed: "3V3 rail >= 500mA peak-capable"
- note removed: "40 MHz XTAL: CL=(C1×C2)/(C1+C2)+Cstray. Start C1=C2=16 pF for CL=10 pF, Cstray=2 pF; L2=24 nH initial. Measure/tune to ±10 ppm."
- note removed: "BQ25611D NVDC: /CE defaults HIGH (charge off); firmware sets 180 mA ICHG and source-aware IINDPM before enable. 1S raw cell: 18650 default / 21700 alternate; welded-tab leads only; BQ298217 + CSD87313DMS independent protection."
- note removed: "Barometer"
- note removed: "Boot Button"
- note removed: "C1=C2=2*(CL-Cstray) For CL=10pF and Cstray about 2pF: start at 16pF; measure and tune."
- note removed: "Charger, Battery Protection & Gauge"
- note removed: "Crystals"
- note removed: "Decoupling Capacitors (MCU)"
- note removed: "EXTERNAL W25Q128JVSIQ (16 MB) — keep bus short and matched."
- note removed: "HSE / LSE"
- note removed: "I2C 7-bit: 0x30 (fixed; CS high) CAP: >=10u low-ESR; keep high-current traces away."
- note removed: "I2C 7-bit: 0x46 (SDO=Earth; CSB high) No copper/vias below pressure port."
- note removed: "I2C 7-bit: 0x47 (ADDR=Earth)"
- note removed: "I2C 7-bit: 0x4E (normal mode)"
- note removed: "I2C 7-bit: 0x55 (fixed)"
- note removed: "I2C 7-bit: 0x6B (fixed)"
- note removed: "IM73A135 VDD is 2.75V MICBIAS; place C51/C52 at the mic. Configure ADC IN1 impedance to 20k; C55/C59 + R39/R43 form matched AC-coupled differential paths. Keep OUT+/OUT- differential and matched."
- note removed: "Impact Sensor"
- note removed: "JTAG / Recovery"
- note removed: "JTAG recovery: GPIO39–42. UART0: GPIO43/44. Native USB Serial/JTAG remains on GPIO19/20."
- note removed: "Layout: both sensors on rigid board. Place IIS3DWB10IS near the cue-front rigid insert, preserve documented axis orientation, keep SPI routes short, and do not soft-mount."
- note removed: "Layout: crystal and caps tight to pins; uninterrupted RF ground; antenna at board edge with CA-C03 keepout; no copper/traces in antenna keepout."
- note removed: "MCU ESP32-S3R8"
- note removed: "Magnetometer"
- note removed: "Main Motion IMU"
- note removed: "Microphone"
- note removed: "Mode: QuadSPI"
- note removed: "NOR FLASH"
- note removed: "NP = Normal P = Directly in Flash"
- note removed: "PI Filter Antenna"
- note removed: "Place R5/R6 close to the MCU USB pins."
- note removed: "Pull-Up"
- note removed: "R8 in-package 8 MB octal PSRAM reserves SPICS1 and GPIO33–GPIO37. Pins are intentionally labeled INTERNAL and are not routed to peripherals."
- note removed: "REFCLK, DBG1, RES14/15 to ground; DBG2 NC. REG gets 100 nF; VDD/VDDIO each 100 nF + 1 uF bulk. Series pads are TUNE."
- note removed: "RF PATH: ESP32 C-L-C -> low-C ESD -> CA-C03 0R/3nH/0R. All values TUNE; final PCB/enclosure VNA + OTA validation is required."
- note removed: "RF Voltage Filter"
- note removed: "RGB Status LED"
- note removed: "RST Button"
- note removed: "SPI Mode 1: SDx/SCx tied to VDDIO; auxiliary pins NC; CS high. VDD/VDDIO 100 nF + 1 uF bulk. Series pads are TUNE."
- note removed: "Status LEDs"
- note removed: "TPS22919 gates the 1M/330k battery ADC divider (no continuous drain). QOD discharges BAT_ADC_SENSE when off; VPACK=VADC x 4.0303. Firmware: wait >=125 ms after BAT_ADC_EN before sampling."
- note removed: "USB_C"
- note removed: "VBUS + 3V3"
- note removed: "VSYS -> +3V3"
- note removed: "Voltage Converter"
- note removed: "WS2812-2020"
- note removed: "Z=(35+j10)R"
- note removed: "Z=50R"
