File: PCB/CueTracker/rear_main.kicad_sch (KiCad schematic)
At the start: 134 parts, among them J1 USB4105-GF-A, J101 FH34SRJ-24S-0.5SH(50), J102 FH34SRJ-8S-0.5SH(50), Q1 CSD87313DMS, Q2 2N7002-7-F, SW1 SHIP EXIT, U1 TUSB320LAI, U10 BQ298217, U13 TLV320ADC6120IRTER, U14 BQ27427, U16 TPS22919DCKR, U17 TPS259470A, U18 TPD2E2U06DCKR, U19 SN74LVC1G17DBVR, U2 USBLC6-2SC6, U3 ESP32-S3-PICO-1-N8R8, U5 TPS63802DLAR, U7 BQ25611D, U9 TPS22919, Y2 FC-135R 32.768kHz 7pF

Commit message: pcb: clean up CueTracker split
Parts:
- removed C34: 100n, Capacitor_SMD:C_0402_1005Metric, symbol Device:C_Small
- removed D3: ESD441DPYR, CueTracker_Exact:TI_DPY0002A_X1SON2_1.0x0.6mm, symbol CueTracker_Exact:ESD441DPYR
- removed R62: 0R, Resistor_SMD:R_0603_1608Metric, symbol Device:R_Small
- removed TP20: ADC_CH2_P, TestPoint:TestPoint_Pad_D1.0mm, symbol Connector:TestPoint
- removed TP21: ADC_CH2_N, TestPoint:TestPoint_Pad_D1.0mm, symbol Connector:TestPoint
- removed U18: TPD2E2U06DCKR, CueTracker_Exact:TI_DCK0003A_SC70-3_2.0x1.25mm_P0.65mm, symbol CueTracker_Exact:TPD2E2U06DCKR
- added C44, C45: 100n, Capacitor_SMD:C_0402_1005Metric, symbol Device:C_Small
- added C46, C47: 1u, Capacitor_SMD:C_0603_1608Metric, symbol Device:C_Small
- added D4: ESD441DPYR, CueTracker_Exact:TI_DPY0002A_X1SON2_1.0x0.6mm, symbol Diode:ESD5Zxx
- added MK2: IM73A135V01, Sensor_Audio:Infineon_PG-LLGA-5-2, symbol Sensor_Audio:IM73A135V01
- added R36, R37: 0R, Resistor_SMD:R_0603_1608Metric, symbol Device:R_Small
- added U3: TPD2E2U06DCKR, CueTracker_Exact:TI_DCK0003A_SC70-3_2.0x1.25mm_P0.65mm, symbol Power_Protection:TPD2E2U06DCK
- C12: now not fitted
- JP1: Assembly Mutually exclusive with U14; controlled heavy solder or cop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 -> Mutually exclusive with U13; controlled heavy solder or cop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; Current_Rating 3 A normal minimum; validate protector fault transient -> 3 A normal minimum when populated; Notes Mutually exclusive with U14 integrated current path -> Mutually exclusive bypass for a no-gauge/high-current servi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; Population Populate default R0_3A only -> DNP default; fit only when U13 is omitted; now not fitted
- MK1: Channel (none) -> ADC channel 1 differential input; MPN (none) -> IM73A135V01XTSA1; Manufacturer (none) -> Infineon Technologies; Package (none) -> PG-LLGA-5-2; Population (none) -> Populate
- U10: renamed from U13; Audio_Channels (none) -> MK1 to IN1P/IN1M; MK2 to IN2P/IN2M; shared MICBIAS
- U13: renamed from U14; Assembly (none) -> Mutually exclusive with JP1; Current_Limit 2 A long-term RMS maximum -> 2 A long-term RMS maximum per TI; Notes Optional gauge variant only; integrated path limited to 2 A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 -> Default fuel-gauge path for sub-2 A RMS operation; 3 A is t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; Population DNP default R0_3A; fit only in R0_GAUGE_2A with JP1 open -> Populate default; JP1 must be DNP; now fitted
- renumbered C64 to C1, C19 to C10, C20 to C11, C30 to C14, C31 to C15, C14 to C16, C15 to C17, C16 to C18, C17 to C19, C1 to C2, C18 to C20, C60 to C21, C61 to C22, C62 to C23, C21 to C24, C22 to C25, C23 to C26, C24 to C27, C25 to C28, C27 to C29, C2 to C3, C38 to C30, C39 to C31, C40 to C32, C41 to C33, C42 to C34, C43 to C35, C44 to C36, C45 to C37, C46 to C38, C47 to C39, C3 to C4, C51 to C40, C52 to C41, C55 to C42, C59 to C43, C53 to C48, C56 to C49, C4 to C5, C57 to C50, C58 to C51, C5 to C6, C6 to C7, C7 to C8, C63 to C9, J101 to J2, J102 to J3, L3 to L1, L1 to L2, L2 to L3, Q2 to Q1, Q1 to Q2, R57 to R1, R56 to R10, R8 to R11, R6 to R12, R9 to R13, R10 to R14, R14 to R15, R54 to R17, R17 to R18, R60 to R19, R1 to R2, R18 to R20, R50 to R21, R52 to R22, R53 to R23, R20 to R24, R21 to R25, R51 to R26, R22 to R27, R61 to R28, R59 to R29, R2 to R3, R37 to R30, R39 to R31, R43 to R32, R23 to R33, R25 to R34, R24 to R35, R30 to R38, R31 to R39, R15 to R4, R33 to R40, R44 to R42, R45 to R43, R16 to R5, R3 to R6, R4 to R7, R5 to R8, R55 to R9, TP6 to TP4, TP7 to TP5, TP8 to TP6, TP22 to TP7, TP23 to TP8, U17 to U1, U9 to U11, U10 to U12, U1 to U2, U19 to U4, U2 to U5, U3 to U6, U5 to U7, U16 to U8, U7 to U9, Y2 to Y1
Connections:
- net +3V3_HMI: now also R29.2; no longer R29.1
- net BAT_ADC_SENSE: now also R33.1, C45.1; no longer R33.2
- net Earth: now also C2.2, C44.2, C45.2, D4.2 (A), MK2.4 (GND), MK2.5 (GND), U3.3
- net LCD_BL: now also R29.1; no longer R29.2
- net USB_CC1: now also U3.1
- net USB_CC2: now also U3.2
- net VBUS_RAW: now also D4.1 (K); no longer C2.2
- net at C40.1, C41.1, MK1.2 (V_{DD})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: now also C44.1, MK2.2 (V_{DD})
- net at U11.5 (QOD), U11.6 (VOUT): now also R33.2; no longer R33.1
- net ADC_CH2_N: no longer names the net of U10.4 (IN2M_GPO1)
- net ADC_CH2_N: now also R37.2
- net ADC_CH2_P: no longer names the net of U10.3 (IN2P_GPI1)
- net ADC_CH2_P: now also R36.2
- new net: C46.2, R36.1
- new net: C46.1, MK2.1 (OUT+)
- new net: C47.1, MK2.3 (OUT-)
- new net: C47.2, R37.1
- no-connect marks 19 -> 18
Other:
- note added: "I2C 7-bit: 0x55 (fixed) BQ27427 populated default; JP1 DNP. Gauge path: <=2 A long-term RMS."
- note added: "IM73A135 VDD is 2.75 V MICBIAS; C40 and C44 are the per-microphone 100 nF bypass capacitors and C41 is the shared 1 uF MICBIAS capacitor. MK1 drives ADC IN1P/IN1M and MK2 drives ADC IN2P/IN2M; keep both differential pairs matched. MK2 is populated for R0 and may become DNP after validation. Enclosure: use a sealed external acoustic chimney, isolated from the BMP581 ePTFE atmospheric vent."
- note added: "MCU ESP32-PICO"
- note added: "Microphones"
- note added: "Status LEDs"
- note removed: "ESP32-S3-PICO-1 integrates the 40 MHz crystal, 8 MB flash and 8 MB octal PSRAM; no external flash or 40 MHz crystal network is fitted."
- note removed: "I2C 7-bit: 0x55 (fixed)"
- note removed: "IM73A135 VDD is 2.75 V MICBIAS; place C51/C52 at the microphone. Configure ADC IN1 for the differential microphone path and keep OUT+/OUT- matched. Enclosure: use a sealed external acoustic chimney, isolated from the BMP581 ePTFE atmospheric vent. ADC channel 2 is routed to TP20/TP21 for test or optional expansion."
- note removed: "Microphone"
- note removed: "PICO internal Flash / PSRAM"
- moved on the sheet: AE1, BOOT1, BT1, C1, C10, C11, C13, C14, C15, C16, C17, C18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
